File: Electronics/soi25.kicad_sch (KiCad schematic)
At the start: 17 parts, among them M1 Motor_DC, U1 MPU-9250, U3 DRV8833PW, U4 LM2596S-5

Commit message: Update the pcb and schematic
Parts:
- removed R4, R5: 10k, Resistor_SMD:R_0201_0603Metric, symbol Device:R
- removed U3: DRV8833PW, Package_SO:TSSOP-16_4.4x5mm_P0.65mm, symbol Driver_Motor:DRV8833PW
- added C4, C9: 0.1 uF, Capacitor_SMD:C_0402_1005Metric_Pad0.74x0.62mm_HandSolder, symbol Device:C_Polarized
- added C7: 10 uF, Capacitor_SMD:C_0402_1005Metric_Pad0.74x0.62mm_HandSolder, symbol Device:C_Polarized
- added C8: 10 nF, Capacitor_SMD:C_0402_1005Metric_Pad0.74x0.62mm_HandSolder, symbol Device:C_Polarized
- added U2: DRV8833PWP, Package_SO:HTSSOP-16-1EP_4.4x5mm_P0.65mm_EP3.4x5mm_Mask2.46x2.31mm_ThermalVias, symbol Driver_Motor:DRV8833PWP
- C1: value 680 uF -> 470 uF; footprint Capacitor_SMD:CP_Elec_4x3 -> Capacitor_THT:C_Radial_D4.0mm_H5.0mm_P1.50mm
- C2: value 220 uF -> 330 uF; footprint Capacitor_SMD:CP_Elec_4x3 -> Capacitor_THT:C_Radial_D4.0mm_H5.0mm_P1.50mm
- C3, C5, C6: footprint Capacitor_SMD:CP_Elec_4x3 -> Capacitor_SMD:C_0402_1005Metric_Pad0.74x0.62mm_HandSolder
- R3, R7, R8: footprint Resistor_SMD:R_0201_0603Metric -> Resistor_SMD:R_0402_1005Metric_Pad0.72x0.64mm_HandSolder
Connections:
- net GND: now also U1.20 (RESV_GND), U1.9 (AD0/MISO), C4.2, C7.2, C8.2, C9.2, U2.13 (GND), U2.17 (GND)
- net at A1.17 (3V3), R7.1, R8.2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: now also U1.1 (RESV_VDDIO), U1.22 (~{CS}), C4.1, C8.1; no longer C5.2, C6.1
- net at A1.27 (VUSB/5V), C2.2, L1.2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: now also C5.2, C6.1, C7.1, U2.12 (VM)
- net at U1.10 (REGOUT): now also C9.1
- net at M1.1 (+): now also U2.2 (AOUT1)
- net at M1.2 (-): now also U2.4 (AOUT2)
- net at A1.20 (A1): now also U2.16 (AIN1)
- net at C3.1: now also U2.14 (VINT)
- net at A1.19 (A0): now also U2.1 (~{SLEEP})
- net at A1.21 (A2): now also U2.15 (AIN2)
- net at C5.1: now also U2.11 (VCP)
- net at R3.1: now also U2.3 (AISEN)
